File: kicad_twe_base.kicad_pcb (KiCad board)
At the start: 2 copper layers, 72 x 47.5 mm, 18 parts, among them U1 TWE-L-DP-W

Commit message: 署名等を入れた
Parts:
- added ~: signature_koino, KICAD_MYLIB:signature_koino, F.Cu at (40.6, -45.7)
Other:
- board text added: "TWELITE_BASE"
Changed lines of the file:
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@@
+    )
+  )
+  (footprint "KICAD_MYLIB:signature_koino" (layer "F.Cu")
+    (at 40.64 -45.72)
+    (attr through_hole)
+    (fp_text reference "~" (at 2.54 -3.81) (layer "F.SilkS")
+      (effects (font (size 1 1) (thickness 0.15)))
+    )
+    (fp_text value "signature_koino" (at 6.35 -5.58) (layer "F.Fab")
+      (effects (font (size 1 1) (thickness 0.15)))
+    )
+    (fp_text user "Twitter:@koino_mfg" (at 0 0.4275) (layer "F.SilkS")
+      (effects (font (size 1 1) (thickness 0.1)) (justify left))
     )
   )
@@
     (effects (font (size 1.2 1.2) (thickness 0.1)))
   )
+  (gr_text "TWELITE_BASE" (at 40.64 -43.18) (layer "F.SilkS")
+    (effects (font (size 1 1) (thickness 0.1)) (justify left))
+  )
   (gr_text "VCC" (at 69.7 -10) (layer "F.SilkS")
